Commit message: Align interfaces and TF with the running car; cut Jetson CPU load
- laksa_interfaces: add DriveCommand.brake and VescState brake_active,
  telemetry_sequence and telemetry_age_ms, matching the firmware flashed
  on the ESP32 (the autonomy-handoff fields the supervisor already reads).
- URDF: root the robot at base_footprint. The fused stack publishes
  odom -> base_footprint from the EKF, so rooting at zed_camera_link gave
  base_footprint two TF parents.
- lidar_guard, zed_base_pose_adapter: feed tf2 from /tf_static only instead
  of deserializing every /tf message in Python; the adapter also caches
  its static camera <- base transform.
- scan_quality: vectorize scan statistics with NumPy.
- drive_supervisor: take the scan and ZED cloud as raw bytes, since they
  are used only as freshness signals.

Measured on the Orin Nano: lidar_guard 37% -> 6%, zed_base_pose_adapter
34% -> 5%, drive_supervisor 55% -> 34% CPU.

Co-Authored-By: Claude Opus 5.5 <noreply@anthropic.com>

File: firmware/esp32-s3/jetson/laksa_description/urdf/laksa_visualization.urdf (robot description, URDF)
Before this commit: robot laksa_visualization, 4 links, 3 joints
Joints:
- removed joint zed_to_base_footprint
- added joint base_footprint_to_zed: type fixed, parent base_footprint, child zed_camera_link, origin xyz=0.108069 0 0.140002 rpy=0 0.06981317007977318 0
